File: ESP32S3-DEVBOARD.kicad_sch (KiCad schematic)
At the start: 56 parts, among them J1 PinHeader_1x22_P2.54mm_Vertic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, J2 PinHeader_1x22_P2.54mm_Vertic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, J3 G-Switch_GT-USB-7010ASV, J4 G-Switch_GT-USB-7010ASV, Q1 BC817-40,215, Q2 BC817-40,215, SW1 TS-1088-AR02016, SW2 TS-1088-AR02016, SW3 TS-1088-AR02016, SW4 TS-1088-AR02016, SW5 SHOU_HAN_1.27-8P_TPPT, U1 AMS1117-3.3, U2 ESP32-S3-WROOM-1, U3 USBLC6-2P6, U4 CP2102N-A02-GQFN28R, U5 BMI270, U6 USBLC6-2P6

Commit message: fixed BOM
Parts:
- C14: MFR.Part # CL10A106MA8NRNC -> (none)
- C3, C6, C8: MFR Part # (none) -> CL10A106MA8NRNC; MFR.Part # CL10A106MA8NRNC -> (none)
- D1, D3: MFR Part # (none) -> 16-213SDRC/S530-A3/TR8; MFR.Part # 16-213SDRC/S530-A3/TR8 -> (none)
- D2, D4: MFR Part # (none) -> 16-213/GHC-YR1S1/3T; MFR.Part # 16-213/GHC-YR1S1/3T -> (none)
- J1, J2, U2: now left out of the parts list
- R1, R5: MFR Part # (none) -> RC0402FR-070RL; Mfr. Part # RC0402FR-070RL -> (none)
- R10: MFR Part # (none) -> 0402WGF4752TCE; Mfr. Part # 0402WGF4752TCE -> (none)
- R11, R12, R20, R21: MFR Part # (none) -> 0402WGF1001TCE; MFR.Part # 0402WGF1001TCE -> (none)
- R13, R14, R15, R2, R3, R4, R8: MFR Part # (none) -> RC0402FR-0710KL; Mfr. Part #  RC0402FR-0710KL -> (none)
- R16, R17, R6, R7: MFR Part # (none) -> 0402WGF5101TCE; MFR.Part # 0402WGF5101TCE -> (none)
- R9: MFR Part # (none) -> FRC0402F2212TS; Mfr. Part #  FRC0402F2212TS -> (none)
- SW1, SW2, SW3, SW4: MFR Part # (none) -> TS-1088-AR02016; Mfr. Part # TS-1088-AR02016 -> (none)
- SW5: LCSC (none) -> C6386921; LCSC Part #  C6386921 -> (none); MFR Part # (none) -> 1.27-8P TPPT; Mfr. Part #  1.27-8P TPPT -> (none)
- U3, U6: MFR Part # (none) -> USBLC6-2P6; Mfr. Part #  USBLC6-2P6 -> (none)
- U5: MFR Part # (none) -> BMI270; Mfr. Part #  BMI270 -> (none)
